Commit message: fixed urdf file for displaying colors correctly. also fixed some link positions to avoid visual glitches on overlaping areas.

File: src/tortoisebot/urdf/tortoisebot.urdf (robot description, URDF)
Before this commit: robot tortoisebot, 6 links, 5 joints
Joints:
- joint front_caster_joint: origin xyz=0.3 0 0 rpy=0 0 0 -> xyz=0.3 0 0.001 rpy=0 0 0
- joint left_wheel_joint: origin xyz=-0.2825 0.125 -.15 rpy=-1.5708 0 0 -> xyz=-0.2825 0.124 -.15 rpy=-1.5708 0 0
- joint right_wheel_joint: origin xyz=-0.2825 -0.125 -.15 rpy=-1.5708 0 0 -> xyz=-0.2825 -0.124 -.15 rpy=-1.5708 0 0

Commit message: fixed movement but some tunnign is still needed

File: src/tortoisebot/urdf/tortoisebot.urdf (robot description, URDF)
Before this commit: robot tortoisebot, 6 links, 5 joints
Joints:
- joint front_caster_joint: origin xyz=0.3 0 0.001 rpy=0 0 0 -> xyz=0.3 0 0 rpy=0 0 0
- joint left_wheel_joint: origin xyz=-0.2825 0.124 -.15 rpy=-1.5708 0 0 -> xyz=-0.2825 0.125 -.15 rpy=-1.5708 0 0
- joint right_wheel_joint: origin xyz=-0.2825 -0.124 -.15 rpy=-1.5708 0 0 -> xyz=-0.2825 -0.125 -.15 rpy=-1.5708 0 0
